File: Pop-In RP2040.kicad_pcb (KiCad board)
At the start: 4 copper layers, 18 x 22 mm, 31 parts, among them U1 RP2040, U2 W25Q32JVXGIQ, Y1 12MHz

Commit message: ...
Parts:
- moved C10 48.3 mm to (100.2, 95.7)
- moved C11 48.3 mm to (99.2, 95.7)
- moved C12 48.3 mm to (101.2, 95.7)
- moved C14 48.3 mm to (102.2, 95.7)
- moved C17 48.3 mm to (100.1, 108.4)
- moved C5 48.3 mm to (94.5, 102.9)
- moved D1 48.3 mm to (95.1, 91.0)
- moved LED1 48.3 mm to (104.4, 95.1)
- moved R1 48.3 mm to (103.1, 108.7)
- moved R2 48.3 mm to (104.4, 108.7)
- moved C13 48.3 mm to (95.1, 95.3)
- moved C16 48.3 mm to (96.2, 108.4)
- moved C4 48.3 mm to (96.2, 97.2)
- moved C6 48.3 mm to (105.7, 102.9)
- moved C8 48.3 mm to (99.8, 106.5)
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
Commit message: ...
Routing:
- net ADC_REF: track 20.1 -> 18.6 mm
- net io29: track 10.2 -> 11.1 mm
- net io9: track 7.06 -> 7.82 mm

Commit message: Seriously messin' with 3D
Changed lines of the file:
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@@
       ) (layer "B.SilkS") (width 0) (fill solid))
   )
-  (gr_text "This is not a\nrPI Pico\nBut\nit works like one" (at 106.35516 96.212877 90) (layer "B.SilkS")
+  (gr_text "This is not a rPI Pico\nBut\nit works like one" (at 106.638284 98.605787 90) (layer "B.SilkS")
     (effects (font (size 0.4 0.4) (thickness 0.1)) (justify mirror))
   )
@@
   (segment (start 92.044624 99.365) (end 92.276471 99.596847) (width 0.2) (layer "F.Cu") (net 8))
   (segment (start 92.276471 100.360099) (end 94.155207 102.238835) (width 0.2) (layer "F.Cu") (net 8))
+  (segment (start 95.256523 103.473165) (end 92.796621 103.473165) (width 0.2) (layer "F.Cu") (net 9))
   (segment (start 91.004112 100.62551) (end 90.994622 100.635) (width 0.2) (layer "F.Cu") (net 9))
-  (segment (start 95.256523 103.473165) (end 93.529453 103.473165) (width 0.2) (layer "F.Cu") (net 9))
+  (segment (start 92.210271 101.506953) (end 92.210271 100.859585) (width 0.2) (layer "F.Cu") (net 9))
   (segment (start 91.009431 100.620191) (end 90.994622 100.635) (width 0.2) (layer "F.Cu") (net 9))
+  (segment (start 92.632027 101.928709) (end 92.210271 101.506953) (width 0.2) (layer "F.Cu") (net 9))
+  (segment (start 92.796621 103.473165) (end 92.632027 103.308571) (width 0.2) (layer "F.Cu") (net 9))
+  (segment (start 92.632027 103.308571) (end 92.632027 101.928709) (width 0.2) (layer "F.Cu") (net 9))
   (segment (start 92.210271 100.859585) (end 91.976196 100.62551) (width 0.2) (layer "F.Cu") (net 9))
-  (segment (start 96.647122 103.038835) (end 95.690853 103.038835) (width 0.2) (layer "F.Cu") (net 9))
-  (segment (start 93.070008 103.013719) (end 93.070008 103.006019) (width 0.2) (layer "F.Cu") (net 9))
-  (segment (start 92.618631 102.554643) (end 92.618631 101.915313) (width 0.2) (layer "F.Cu") (net 9))
-  (segment (start 92.618631 101.915313) (end 92.210271 101.506953) (width 0.2) (layer "F.Cu") (net 9))
-  (segment (start 93.529453 103.473165) (end 93.070008 103.013719) (width 0.2) (layer "F.Cu") (net 9))
-  (segment (start 92.210271 101.506953) (end 92.210271 100.859585) (width 0.2) (layer "F.Cu") (net 9))
   (segment (start 91.976196 100.62551) (end 91.004112 100.62551) (width 0.2) (layer "F.Cu") (net 9))
   (segment (start 95.690853 103.038835) (end 95.256523 103.473165) (width 0.2) (layer "F.Cu") (net 9))
-  (segment (start 93.070008 103.006019) (end 92.618631 102.554643) (width 0.2) (layer "F.Cu") (net 9))
+  (segment (start 96.647122 103.038835) (end 95.690853 103.038835) (width 0.2) (layer "F.Cu") (net 9))
+  (segment (start 95.422209 103.873165) (end 92.630935 103.873165) (width 0.2) (layer "F.Cu") (net 10))
+  (segment (start 92.042632 101.905) (end 90.994622 101.905) (width 0.2) (layer "F.Cu") (net 10))
+  (segment (start 95.856539 103.438835) (end 95.422209 103.873165) (width 0.2) (layer "F.Cu") (net 10))
+  (segment (start 96.647122 103.438835) (end 95.856539 103.438835) (width 0.2) (layer "F.Cu") (net 10))
+  (segment (start 92.219714 102.608202) (end 92.218631 102.607119) (width 0.2) (layer "F.Cu") (net 10))
+  (segment (start 92.219714 103.461944) (end 92.219714 102.608202) (width 0.2) (layer "F.Cu") (net 10))
+  (segment (start 95.85654 103.438835) (end 96.647122 103.438835) (width 0.2) (layer "F.Cu") (net 10))
+  (segment (start 92.218631 102.607119) (end 92.218631 102.080999) (width 0.2) (layer "F.Cu") (net 10))
   (segment (start 92.218631 102.080999) (end 92.042632 101.905) (width 0.2) (layer "F.Cu") (net 10))
-  (segment (start 96.647122 103.438835) (end 95.856539 103.438835) (width 0.2) (layer "F.Cu") (net 10))
-  (segment (start 93.363768 103.873165) (end 92.715521 103.224918) (width 0.2) (layer "F.Cu") (net 10))
-  (segment (start 95.85654 103.438835) (end 96.647122 103.438835) (width 0.2) (layer "F.Cu") (net 10))
-  (segment (start 92.670008 103.179405) (end 92.715521 103.224918) (width 0.2) (layer "F.Cu") (net 10))
-  (segment (start 92.042632 101.905) (end 90.994622 101.905) (width 0.2) (layer "F.Cu") (net 10))
-  (segment (start 95.422209 103.873165) (end 93.363768 103.873165) (width 0.2) (layer "F.Cu") (net 10))
-  (segment (start 92.670008 103.171705) (end 92.670008 103.179405) (width 0.2) (layer "F.Cu") (net 10))
-  (segment (start 92.218631 102.720328) (end 92.218631 102.080999) (width 0.2) (layer "F.Cu") (net 10))
-  (segment (start 92.670008 103.171705) (end 92.218631 102.720328) (width 0.2) (layer "F.Cu") (net 10))
-  (segment (start 95.856539 103.438835) (end 95.422209 103.873165) (width 0.2) (layer "F.Cu") (net 10))
-  (segment (start 92.270008 103.345091) (end 92.270008 103.337391) (width 0.2) (layer "F.Cu") (net 11))
+  (segment (start 92.630935 103.873165) (end 92.219714 103.461944) (width 0.2) (layer "F.Cu") (net 10))
   (segment (start 96.647122 103.838835) (end 96.022225 103.838835) (width 0.2) (layer "F.Cu") (net 11))
-  (segment (start 93.198082 104.273165) (end 92.270008 103.345091) (width 0.2) (layer "F.Cu") (net 11))
-  (segment (start 92.107617 103.175) (end 90.994622 103.175) (width 0.2) (layer "F.Cu") (net 11))
-  (segment (start 95.587895 104.273165) (end 93.198082 104.273165) (width 0.2) (layer "F.Cu") (net 11))
-  (segment (start 92.270008 103.337391) (end 92.107617 103.175) (width 0.2) (layer "F.Cu") (net 11))
   (segment (start 96.022225 103.838835) (end 95.587895 104.273165) (width 0.2) (layer "F.Cu") (net 11))
+  (segment (start 95.587895 104.273165) (end 92.465249 104.273165) (width 0.2) (layer "F.Cu") (net 11))
+  (segment (start 91.367084 103.175) (end 90.994622 103.175) (width 0.2) (layer "F.Cu") (net 11))
+  (segment (start 92.465249 104.273165) (end 91.367084 103.175) (width 0.2) (layer "F.Cu") (net 11))
+  (segment (start 93.029094 104.676467) (end 91.226089 104.676467) (width 0.2) (layer "F.Cu") (net 12))
+  (segment (start 93.032396 104.673165) (end 93.029094 104.676467) (width 0.2) (layer "F.Cu") (net 12))
+  (segment (start 91.226089 104.676467) (end 90.994622 104.445) (width 0.2) (layer "F.Cu") (net 12))
   (segment (start 96.212792 104.673165) (end 93.032396 104.673165) (width 0.2) (layer "F.Cu") (net 12))
   (segment (start 96.647122 104.238835) (end 96.212792 104.673165) (width 0.2) (layer "F.Cu") (net 12))
-  (segment (start 92.804231 104.445) (end 90.994622 104.445) (width 0.2) (layer "F.Cu") (net 12))
-  (segment (start 93.032396 104.673165) (end 92.804231 104.445) (width 0.2) (layer "F.Cu") (net 12))
   (segment (start 92.525805 105.413835) (end 92.22464 105.715) (width 0.2) (layer "F.Cu") (net 13))
   (segment (start 97.484622 105.076335) (end 97.147122 105.413835) (width 0.2) (layer "F.Cu") (net 13))
@@
   (via (at 105.401569 107.644144) (size 0.4) (drill 0.3) (layers "F.Cu" "B.Cu") (free) (net 33))
   (via (at 100.721603 101.646042) (size 0.4) (drill 0.3) (layers "F.Cu" "B.Cu") (remove_unused_layers) (free) (net 33))
-  (via (at 93.644548 102.555742) (size 0.3) (drill 0.2) (layers "F.Cu" "B.Cu") (remove_unused_layers) (free) (net 33))
+  (via (at 93.259121 102.505449) (size 0.3) (drill 0.2) (layers "F.Cu" "B.Cu") (remove_unused_layers) (free) (net 33))
   (via (at 102.573111 101.683514) (size 0.3) (drill 0.2) (layers "F.Cu" "B.Cu") (free) (net 33))
   (via (at 107.075116 102.861066) (size 0.3) (drill 0.2) (layers "F.Cu" "B.Cu") (remove_unused_layers) (free) (net 33))
