File: test3.kicad_pcb (KiCad board)
At the start: 2 copper layers, 30.5 x 36.6 mm, 1 part

Commit message: ...
Other:
- board text added: "Poke da Bunny!"
- board text removed: "Poke da Rabbit!"
Changed lines of the file:
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@@
     (pad_to_mask_clearance 0)
     (pcbplotparams
-      (layerselection 0x00010fc_ffffffff)
+      (layerselection 0x0000030_7ffffffe)
       (disableapertmacros false)
       (usegerberextensions false)
@@
       (hpglpendiameter 15.000000)
       (dxfpolygonmode true)
-      (dxfimperialunits true)
+      (dxfimperialunits false)
       (dxfusepcbnewfont true)
       (psnegative false)
@@
       (sketchpadsonfab false)
       (subtractmaskfromsilk false)
-      (outputformat 1)
+      (outputformat 3)
       (mirror false)
-      (drillshape 1)
+      (drillshape 0)
       (scaleselection 1)
       (outputdirectory "")
@@
       (rotate (xyz 0 0 0))
     )
-    (model "${KIPRJMOD}/3D/turd.step"
+    (model "${KIPRJMOD}/3D/Pop-In RP2040-b.step" hide
+      (offset (xyz -100 101.27 1))
+      (scale (xyz 1 1 1))
+      (rotate (xyz 0 0 0))
+    )
+    (model "${KIPRJMOD}/3D/Pop-In RP2040.step"
       (offset (xyz -100 101.27 1))
       (scale (xyz 1 1 1))
@@
   (gr_line (start 162.56 77.74) (end 162.56 114.3) (layer "Edge.Cuts") (width 0.05))
   (gr_line (start 132.08 77.74) (end 162.56 77.74) (layer "Edge.Cuts") (width 0.05))
-  (gr_text "Poke da\nRabbit!" (at 150.298303 89.988826) (layer "B.SilkS")
+  (gr_text "Poke da\nBunny!" (at 150.298303 89.988826) (layer "B.SilkS")
     (effects (font (size 0.5 0.5) (thickness 0.1)) (justify right mirror))
   )
-  (gr_text "Poke da\nRabbit!" (at 144.490611 89.889549) (layer "F.SilkS")
+  (gr_text "Poke da\nBunny!" (at 144.490611 89.889549) (layer "F.SilkS")
     (effects (font (size 0.5 0.5) (thickness 0.1)) (justify right))
   )
