File: Pop-In RP2040.kicad_sch (KiCad schematic)
At the start: 33 parts, among them Q1 DMG1012T, U1 RP2040, U2 W25Q32JVXGIQ, Y1 12MHz

Commit message: ...
Other:
- company: (none) -> S. A. Miller
- title: (none) -> Pop-In RP2040 Module
Changed lines of the file:
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@@
 (kicad_sch (version 20211123) (generator eeschema)
   (paper "A4")
+  (title_block
+    (title "Pop-In RP2040 Module")
+    (date "2023-07-14")
+    (rev "0.1.0")
+    (company "S. A. Miller")
+  )
   (junction (at 166.37 113.03) (diameter 0) (color 0 0 0 0)
   )
